File: AHsoundbox.kicad_sch (KiCad schematic)
At the start: 41 parts, among them J1 USB_C_Receptacle_PowerOnly_6P, P1 Conn_01x03, Q2 S8550, Q3 S8050, U1 SZY55F2, U2 T25S128, U3 CL4054

Commit message: Add files via upload
Parts:
- added R17: R, symbol Device:R
- added S2: Conn_01x02, symbol Connector_Generic:Conn_01x02
Connections:
- net GND: now also S2.2 (Pin_2)
- net at R1.2, U1.21 (PB1): now also R17.1
- new net: R17.2, S2.1 (Pin_1)
